File: PCB/DVDLaserScanner.kicad_sch (KiCad schematic)
At the start: 0 parts

Commit message: Modify PCB
Parts:
- added P1: USB_C_Plug_USB2.0, symbol Connector:USB_C_Plug_USB2.0
- added R11: 100K, symbol Device:R
- added R12: 100k, symbol Device:R
- added U3: MIC5365-3.3YC5, Package_TO_SOT_SMD:SOT-353_SC-70-5, symbol Regulator_Linear:MIC5365-3.3YC5
Connections:
- net Actuation control block/5V: now also P1.A4 (VBUS), P1.A9 (VBUS), P1.B4 (VBUS), P1.B9 (VBUS)
- net Actuation control block/GND: now also P1.A1 (GND), P1.A12 (GND), P1.B1 (GND), P1.B12 (GND), P1.S1 (SHIELD), U3.2 (GND)
- new net: R11.1, R12.1, U3.5 (VOUT)
- new net Actuation control block/FOCUS_VCM_I2C_SCL: R11.2
- new net Actuation control block/FOCUS_VCM_I2C_SDA: R12.2
- new net Controller/5V: U3.1 (VIN), U3.3 (EN)
- no-connect marks 0 -> 4
Other:
- sheet Optical Pickup Unit renamed Sanyo HD-850 OPU
- sheet Actuation control block ports: added FOCUS_VCM_I2C_SCL, FOCUS_VCM_I2C_SDA, T+, TRACK_VCM_I2C_SCL, TRACK_VCM_I2C_SDA; removed FOCUS_CTL
- sheet Controller ports: added -5V, DIO_0, DIO_1, DIO_10, DIO_11, DIO_12, DIO_13, DIO_14, DIO_15, DIO_2, DIO_3, DIO_4, DIO_5, DIO_6, DIO_7, DIO_8, DIO_9, TRIG1, TRIG2; removed none
- sheet Emission control block ports: added LD_LOW_SIDE; removed LD_DVD
- sheet Sanyo HD-850 OPU ports: added CD-LD, E, F, HIGH_FREQUENCY_MODE_EN, T+, T-, VR-CD, VR-DVD; removed none
- sheet Sensing block ports: added -5V; removed none
- note added: "Focus: +1.1 mm / -0.7 mm 0.80 mm/V @ 5Hz(positiv = aproach disk) 2.20 um/V @ 1kHz(positiv = aproach disk) Tracking: ±0.4 mm 0.60 mm/V @ 5Hz(positv = periphery of disk) 1.62 um/V @ 1kHz(positv = periphery of disk) Imax 220 mA per motor"
- note added: "I2C pullup resistors"
- note added: "Unused OPU I/O"
- note added: "Unused controller I/O"
- note removed: "1.375V / -0.875V 1/1.8181 ±0.67 V / 1/3.7313"
- note removed: "CD/DVD_SW LASER H UV (CD) L RED (DVD)"
- note removed: "Focus: +1.1 mm / -0.7 mm 0.80 mm/V (positiv = aproach disk) Tracking: ±0.4 mm 0.60 mm/V (positv = periphery of disk) Imax 220 mA"
