File: PCB/controller.kicad_sch (KiCad schematic)
At the start: 1 part, among them J1 Conn_02x15_Row_Letter_First

Commit message: Modify PCB
Connections:
- net -5V: now reaches J1.b4 (Pin_b4)
- no-connect marks 1 -> 0
