File: PCB/emission.kicad_sch (KiCad schematic)
At the start: 6 parts, among them Q1 Q_NMOS_GDS, U1 TLC2274

Commit message: Modify PCB
Parts:
- removed Q1: Q_NMOS_GDS, TO_SOT_Packages_SMD:TO-252-2Lead, symbol DVDLaserScanner-rescue:Q_NMOS_GDS
- removed U1: TLC2274, symbol DVDLaserScanner-rescue:TLC2274
- added Q1: BSS138, Package_TO_SOT_SMD:SOT-23, symbol Transistor_FET:BSS138
- added U5: MCP6022, symbol Amplifier_Operational:MCP6022
Connections:
- net 5V: now also U5.8 (V+)
- net GND: now also U5.4 (V-)
- net INTENSITY: now also U5.3 (+)
- net at R7.1: now also Q1.1 (G)
- net at C4.1, R7.2: now also U5.1
- net at C4.2, R9.2: now also U5.2 (-)
- net at R10.2, R9.1: now also Q1.2 (S)
- new net LD_LOW_SIDE: Q1.3 (D)
