File: PCB/sensing.kicad_sch (KiCad schematic)
At the start: 37 parts, among them U1 TLC2274, U6 TLC2274, U9 TLC2274

Commit message: Modify PCB
Connections:
- net GND: now also C10.2, C2.1, C9.2, R22.1, U9.10 (+), U9.12 (+), U9.3 (+), U9.5 (+); no longer U6.11 (VDD-), U9.11 (VDD-)
- net VC(VREF): no longer C10.2, C2.1, C9.2, R22.1, U9.10 (+), U9.12 (+), U9.3 (+), U9.5 (+)
- new net -5V: U6.11 (VDD-), U9.11 (VDD-)
Changed lines of the file:
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@@
-	)
-	(label "VC(VREF)"
-		(at 266.7 86.36 0)
-		(fields_autoplaced yes)
-		(effects
-			(font
-				(size 1.524 1.524)
-			)
-			(justify left bottom)
-		)
 	)
 	(label "VC(VREF)"
@@
 	(label "PD_BD"
 		(at 204.47 149.86 0)
-		(fields_autoplaced yes)
-		(effects
-			(font
-				(size 1.524 1.524)
-			)
-			(justify left bottom)
-		)
-	)
-	(label "VC(VREF)"
-		(at 266.7 48.26 0)
 		(fields_autoplaced yes)
 		(effects
@@
 		)
 	)
+	(hierarchical_label "GND"
+		(shape input)
+		(at 266.7 86.36 0)
+		(fields_autoplaced yes)
+		(effects
+			(font
+				(size 1.524 1.524)
+			)
+			(justify left)
+		)
+	)
 	(hierarchical_label "A_SIG"
 		(shape input)
@@
 		)
 	)
+	(hierarchical_label "-5V"
+		(shape input)
+		(at 139.7 45.72 180)
+		(fields_autoplaced yes)
+		(effects
+			(font
+				(size 1.524 1.524)
+			)
+			(justify right)
+		)
+	)
 	(hierarchical_label "PD_CHAIN"
 		(shape output)
@@
 		)
 	)
+	(hierarchical_label "D_SIG"
+		(shape input)
+		(at 266.7 26.67 0)
+		(fields_autoplaced yes)
+		(effects
+			(font
+				(size 1.524 1.524)
+			)
+			(justify left)
+		)
+	)
+	(hierarchical_label "D_SIG"
+		(shape input)
+		(at 218.44 119.38 0)
+		(fields_autoplaced yes)
+		(effects
+			(font
+				(size 1.524 1.524)
+			)
+			(justify left)
+		)
+	)
+	(hierarchical_label "RF"
+		(shape input)
+		(at 85.09 57.15 0)
+		(fields_autoplaced yes)
+		(effects
+			(font
+				(size 1.524 1.524)
+			)
+			(justify left)
+		)
+	)
+	(hierarchical_label "B_SIG"
+		(shape input)
+		(at 218.44 106.68 0)
+		(fields_autoplaced yes)
+		(effects
+			(font
+				(size 1.524 1.524)
+			)
+			(justify left)
+		)
+	)
+	(hierarchical_label "5V"
+		(shape input)
+		(at 184.15 81.28 180)
+		(fields_autoplaced yes)
+		(effects
+			(font
+				(size 1.524 1.524)
+			)
+			(justify right)
+		)
+	)
+	(hierarchical_label "-5V"
+		(shape input)
+		(at 184.15 68.58 180)
+		(fields_autoplaced yes)
+		(effects
+			(font
+				(size 1.524 1.524)
+			)
+			(justify right)
+		)
+	)
+	(hierarchical_label "C_SIG"
+		(shape input)
+		(at 266.7 64.77 0)
+		(fields_autoplaced yes)
+		(effects
+			(font
+				(size 1.524 1.524)
+			)
+			(justify left)
+		)
+	)
 	(hierarchical_label "GND"
 		(shape input)
-		(at 184.15 68.58 180)
-		(fields_autoplaced yes)
-		(effects
-			(font
-				(size 1.524 1.524)
-			)
-			(justify right)
-		)
-	)
-	(hierarchical_label "D_SIG"
-		(shape input)
-		(at 266.7 26.67 0)
-		(fields_autoplaced yes)
-		(effects
-			(font
-				(size 1.524 1.524)
-			)
-			(justify left)
-		)
-	)
-	(hierarchical_label "D_SIG"
-		(shape input)
-		(at 218.44 119.38 0)
-		(fields_autoplaced yes)
-		(effects
-			(font
-				(size 1.524 1.524)
-			)
-			(justify left)
-		)
-	)
-	(hierarchical_label "RF"
-		(shape input)
-		(at 85.09 57.15 0)
-		(fields_autoplaced yes)
-		(effects
-			(font
-				(size 1.524 1.524)
-			)
-			(justify left)
-		)
-	)
-	(hierarchical_label "B_SIG"
-		(shape input)
-		(at 218.44 106.68 0)
-		(fields_autoplaced yes)
-		(effects
-			(font
-				(size 1.524 1.524)
-			)
-			(justify left)
-		)
-	)
-	(hierarchical_label "5V"
-		(shape input)
-		(at 184.15 81.28 180)
-		(fields_autoplaced yes)
-		(effects
-			(font
-				(size 1.524 1.524)
-			)
-			(justify right)
-		)
-	)
-	(hierarchical_label "C_SIG"
-		(shape input)
-		(at 266.7 64.77 0)
-		(fields_autoplaced yes)
-		(effects
-			(font
-				(size 1.524 1.524)
-			)
-			(justify left)
-		)
-	)
-	(hierarchical_label "GND"
-		(shape input)
-		(at 139.7 45.72 180)
-		(fields_autoplaced yes)
-		(effects
-			(font
-				(size 1.524 1.524)
-			)
-			(justify right)
-		)
-	)
+		(at 266.7 48.26 0)
+		(fields_autoplaced yes)
+		(effects
+			(font
+				(size 1.524 1.524)
+			)
+			(justify left)
+		)
+	)
